File: src/Model-S.kicad_pcb (KiCad board)
At the start: 2 copper layers, 112.6 x 42.6 mm, 41 parts, among them J1 USB_C_Receptacle, J2 USBFeedThrough, J3 I/O Pin Headers, J4 I/O Screw Terminals, J5 Brook Header, J6 Debug, J7 USB4Pin, J8 ICSP, Q1 BSS138, SW2 SW_PUSH, U1 TPS61240, U2 TS3USB30E, U3 ATmega32U4-AU, X1 XTAL_GND

Commit message: Model S 2.1
Parts:
- removed the G*** at (95.8, 110.3)
- added G***: LOGO, Footprints:logo, F.Cu at (91.7, 110.1)
- added G***: LOGO, Footprints:logo, F.Cu at (137.2, 120.4)
- C1, C10, C11, C12, C2, C3, C4, C5, C6, C7, C8, C9: footprint Capacitor_SMD:C_0805_2012Metric_Pad1.15x1.40mm_HandSolder -> Model_S:C_0805_2012Metric_Pad1.18x1.45mm_HandSolder
- D1, D2: footprint Diode_SMD:D_SOD-123 -> Model_S:D_SOD-123
- J1: footprint typec:Wurth-632723300011 -> Model_S:Shou Han Type-C 24P QCHT
- J2: footprint digikey-footprints:USB_A_Female_UE27AC54100 -> Model_S:USB_A_Female_UE27AC54100
- J3: footprint Connector_PinHeader_2.54mm:PinHeader_2x23_P2.54mm_Vertical -> Model_S:PinHeader_2x23_P2.54mm_Vertical
- J4: footprint GCPCBFootprints:24PinScrewTerminal -> Model_S:24PinScrewTerminal
- J5: footprint Connector_PinHeader_2.54mm:PinHeader_2x10_P2.54mm_Vertical -> Model_S:PinHeader_2x10_P2.54mm_Vertical
- J6: footprint Connector_PinHeader_2.54mm:PinHeader_1x06_P2.54mm_Vertical -> Model_S:PinHeader_1x06_P2.54mm_Vertical
- J7: footprint Connector_PinHeader_2.54mm:PinHeader_1x04_P2.54mm_Vertical -> Model_S:PinHeader_1x04_P2.54mm_Vertical
- J8: footprint Connector_PinHeader_2.54mm:PinHeader_2x03_P2.54mm_Vertical -> Model_S:PinHeader_2x03_P2.54mm_Vertical
- L1: footprint Inductor_SMD:L_0805_2012Metric_Pad1.15x1.40mm_HandSolder -> Model_S:L_0805_2012Metric_Pad1.15x1.40mm_HandSolder
- Q1: footprint Package_TO_SOT_SMD:SOT-23 -> Model_S:SOT-23
- R1, R2, R3, R4, R5, R6, R7: footprint Resistor_SMD:R_0805_2012Metric_Pad1.15x1.40mm_HandSolder -> Model_S:R_0805_2012Metric_Pad1.20x1.40mm_HandSolder
- SW2: footprint Button_Switch_SMD:SW_SPST_TL3342 -> Model_S:SW_SPST_TL3342
- U1: footprint GCPCBFootprints:TPS61240 -> Model_S:TPS61240
- U2: footprint Package_SO:VSSOP-10_3x3mm_P0.5mm -> Model_S:VSSOP-10_3x3mm_P0.5mm
- U3: footprint Package_QFP:TQFP-44_10x10mm_P0.8mm -> Model_S:TQFP-44_10x10mm_P0.8mm
- X1: footprint Crystal:Crystal_SMD_TXC_7M-4Pin_3.2x2.5mm -> Model_S:Crystal_SMD_TXC_7M-4Pin_3.2x2.5mm
- moved C12 8.95 mm to (147.9, 121.3), turned to 0 degrees
- moved U2 3.69 mm to (153.2, 118.7), turned to 180 degrees
- moved R2 1.30 mm to (136.2, 121.6)
- moved Q1 1.30 mm to (138.9, 121.6)
- moved R3 1.30 mm to (141.6, 121.6)
- moved R4 1.08 mm to (114.5, 110.8)
- moved R5 0.78 mm to (114.5, 113.0)
- moved C1 0.41 mm to (128.8, 118.3)
- moved C2 0.41 mm to (125.2, 121.4)
- moved L1 0.41 mm to (132.7, 120.7)
- moved U1 0.41 mm to (128.9, 121.9)
- moved C3 0.36 mm to (108.8, 107.6)
Connections:
- J2 pad 1: VBUS -> +5V
- J5 pad 19: VBUS -> +5V
- J5 pad 20: VBUS -> +5V
- J7 pad 1: VBUS -> +5V
Routing:
- net +5V: track 141.1 -> 226.6 mm, vias 6 -> 10
- net VBUS: track 160.5 -> 108.7 mm
- net D1-: track 63.1 -> 37.8 mm, vias 2 -> 0
- net 3V3NXX: track 85.0 -> 105.6 mm
- net D-: track 42.7 -> 24.5 mm, vias 6 -> 1
- net D11: track 63.9 -> 77.4 mm
- net D14_MISO: track 178.4 -> 170.8 mm, vias 1 -> 0
- net D1+: track 43.3 -> 49.3 mm, vias 2 -> 0
- net GND: track 87.8 -> 93.6 mm, vias 93 -> 98
- net D16_MOSI: track 179.6 -> 174.3 mm, vias 1 -> 0
- net D15_SCK: track 176.5 -> 172.3 mm, vias 1 -> 0
- net D+: track 30.7 -> 26.8 mm, vias 5 -> 1
- net D2-: track 54.6 -> 58.4 mm, vias 1 -> 0
- net GC-D3V: track 38.6 -> 42.4 mm
- net A5: track 97.7 -> 95.0 mm, vias 2 -> 1
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Other:
- rule pad_to_mask_clearance: 0.051 -> 0
- board text added: "Crane Model S"
- board text added: "J1"
- board text added: "J10"
- board text added: "J11"
- board text added: "J12"
- board text added: "J13"
- board text added: "J14"
- board text added: "JLCJLCJLCJLC"
- board text added: "Model S v2.1 Designed by Matt Crane in 2020 Assembled in 2021"
- board text added: "Screw Terminal"
- board text added: "USB-A"
- board text added: "craneslab.xyz"
- board text added: "v2.1"
- board text removed: "v2.0"

Commit message: Model S 2.2
Parts:
- removed the J6 at (116.5, 107.7)
- added ?: , , F.Cu at (144.8, 109.0)
- added ?: , , F.Cu at (129.5, 109.0)
- added C3: 22uF, Model_S:C_0805_2012Metric_Pad1.18x1.45mm_HandSolder, F.Cu at (120.6, 114.5)
- added C4: 22uF, Model_S:C_0805_2012Metric_Pad1.18x1.45mm_HandSolder, F.Cu at (120.6, 116.5)
- added C5: 22uF, Model_S:C_0805_2012Metric_Pad1.18x1.45mm_HandSolder, F.Cu at (120.6, 118.4)
- added R1: 402k, Model_S:R_0805_2012Metric_Pad1.20x1.40mm_HandSolder, F.Cu at (125.6, 113.8)
- added R2: 100k, Model_S:R_0805_2012Metric_Pad1.20x1.40mm_HandSolder, F.Cu at (125.6, 110.0)
- C1: value 2.2uF -> 22uF
- C2: value 4.7uF -> 10nF
- J1: value USB_C_Receptacle -> USB-C Port; footprint Model_S:Shou Han Type-C 24P QCHT -> Project_Pico:Crane_USBC
- L1: footprint Model_S:L_0805_2012Metric_Pad1.15x1.40mm_HandSolder -> Inductor_SMD:L_1008_2520Metric
- U1: value TPS61240 -> TPS61230DRC; footprint Model_S:TPS61240 -> Package_SON:Texas_S-PVSON-N10_ThermalVias
- moved L1 18.2 mm to (118.4, 109.3)
- moved U1 12.4 mm to (122.3, 111.4)
- moved C1 11.8 mm to (122.6, 108.3)
- moved D1 3.90 mm to (120.8, 123.3)
- moved C2 3.89 mm to (124.7, 117.5), turned to 270 degrees
- moved R5 3.47 mm to (149.9, 113.2)
- moved R7 1.66 mm to (113.3, 109.6)
- moved R8 1.66 mm to (113.3, 111.8)
- moved D2 1.17 mm to (120.8, 121.0)
- turned J1 to 0 degrees
- renumbered C7 to C10, C8 to C11, C9 to C12, C10 to C13, C12 to C14, C11 to C15, C3 to C6, C4 to C7, C5 to C8, C6 to C9, J7 to J3, J8 to J4, J3 to J5, J5 to J6, J4 to J7, R2 to R3, R3 to R4, R7 to R5, R1 to R6, R4 to R7, R5 to R8, R6 to R9, SW2 to SW1
Connections:
- C2 pad 1: 5VBoosted -> Net-(C2-Pad1)
- J2 pad 5: GND -> (no net)
- U1 pad 1: GND -> Net-(L1-Pad2)
- U1 pad 2: 5VBoosted -> Net-(L1-Pad2)
- U1 pad 4: 3V3NXX -> 5VBoosted
- U1 pad 5: Net-(L1-Pad2) -> Net-(U1-Pad5)
- U1 pad 6: 3V3NXX -> Net-(C2-Pad1)
- U1 pad 7: (no net) -> Net-(R1-Pad2)
Routing:
- net 3V3NXX: track 105.6 -> 55.7 mm, vias 3 -> 2
- net VBUS: track 108.7 -> 76.1 mm, vias 7 -> 3
- net GC-D3V: track 42.4 -> 18.6 mm, vias 3 -> 1
- net 5VBoosted: track 10.7 -> 28.5 mm, vias 0 -> 3
- net GND: track 93.6 -> 79.5 mm, vias 98 -> 97
- net +5V: track 226.6 -> 215.0 mm, vias 10 -> 9
- net D1+: track 49.3 -> 57.1 mm
- net D1-: track 37.8 -> 43.2 mm
- net Net-(C2-Pad1): track 0.00 -> 4.47 mm
- net Net-(L1-Pad2): track 6.17 -> 2.55 mm
- net Net-(R1-Pad2): track 0.00 -> 3.57 mm
- net D11: track 77.4 -> 73.9 mm, vias 3 -> 2
- net D-: track 24.5 -> 28.0 mm, vias 1 -> 0
- net Net-(R8-Pad1): track 9.30 -> 7.67 mm
- net Net-(R7-Pad1): track 9.92 -> 8.63 mm
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Other:
- board text added: "J8"
- board text added: "Model S"
- board text added: "Model S v2.2 Designed by Matt Crane in 2021 Assembled in 2021"
- board text added: "v2.2"
- board text removed: "3V3NXX"
- board text removed: "Crane Model S"
- board text removed: "GC-D3V"
- board text removed: "Model S v2.1 Designed by Matt Crane in 2020 Assembled in 2021"
- board text removed: "v2.1"

Commit message: Model S 2.3
Parts:
- U2: value TS3USB30E -> TS3USB30ERSWR; footprint Model_S:VSSOP-10_3x3mm_P0.5mm -> Model_S:UQFN-10_1.4x1.8mm_P0.4mm
Connections:
- U2 pad 1: D11 -> D1+
- U2 pad 10: VBUS -> D11
- U2 pad 2: D1+ -> D2+
- U2 pad 3: D2+ -> D+
- U2 pad 4: D+ -> GND
- U2 pad 5: GND -> D-
- U2 pad 6: D- -> D2-
- U2 pad 7: D2- -> D1-
- U2 pad 8: D1- -> GND
- U2 pad 9: GND -> VBUS
Routing:
- net VBUS: track 76.1 -> 84.0 mm
- net GND: track 79.5 -> 85.3 mm, vias 97 -> 96
- net D2+: track 62.8 -> 59.2 mm, vias 0 -> 2
- net D-: track 28.0 -> 31.2 mm
- net D11: track 73.9 -> 76.2 mm
- net D2-: track 58.4 -> 56.1 mm, vias 0 -> 2
- net D1-: track 43.2 -> 44.7 mm
Other:
- board text added: "Model S v2.3 Designed by Matt Crane in 2021 Assembled in 2021"
- board text added: "v2.3"
- board text removed: "Model S v2.2 Designed by Matt Crane in 2021 Assembled in 2021"
- board text removed: "v2.2"
