File: src/Model-S.sch (KiCad schematic (older format))
At the start: 36 parts, among them J1 USB_C_Receptacle, J2 USBFeedThrough, J3 I/O Pin Headers, J4 I/O Screw Terminals, J5 Brook Header, J6 Debug, J7 USB4Pin, J8 ICSP, Q1 BSS138, SW2 SW_PUSH, U1 TPS61240, U2 TS3USB30E, U3 ATmega32U4-AU, X1 XTAL_GND

Commit message: Model S 2.1
Parts:
- C1, C10, C11, C12, C2, C3, C4, C5, C6, C7, C8, C9: footprint Capacitor_SMD:C_0805_2012Metric_Pad1.15x1.40mm_HandSolder -> Model_S:C_0805_2012Metric_Pad1.18x1.45mm_HandSolder; symbol Device:C_Small -> Model-S-rescue:C_Small-Model_S
- D1, D2: footprint Diode_SMD:D_SOD-123 -> Model_S:D_SOD-123; symbol Device:D_Schottky -> Model-S-rescue:D_Schottky-Model_S
- J1: footprint typec:Wurth-632723300011 -> Model_S:Shou Han Type-C 24P QCHT; symbol Model-S-rescue:USB_C_Receptacle-Connector -> Model-S-rescue:USB_C_Receptacle-Model_S
- J2: footprint digikey-footprints:USB_A_Female_UE27AC54100 -> Model_S:USB_A_Female_UE27AC54100; symbol Model-S-rescue:USB_A-Connector -> Model-S-rescue:USB_A-Model_S
- J3: footprint Connector_PinHeader_2.54mm:PinHeader_2x23_P2.54mm_Vertical -> Model_S:PinHeader_2x23_P2.54mm_Vertical; symbol Connector_Generic:Conn_02x23_Odd_Even -> Model-S-rescue:Conn_02x23_Odd_Even-Model_S
- J4: footprint GCPCBFootprints:24PinScrewTerminal -> Model_S:24PinScrewTerminal; symbol Connector_Generic:Conn_01x24 -> Model-S-rescue:Conn_01x24-Model_S
- J5: footprint Connector_PinHeader_2.54mm:PinHeader_2x10_P2.54mm_Vertical -> Model_S:PinHeader_2x10_P2.54mm_Vertical; symbol Connector_Generic:Conn_02x10_Odd_Even -> Model-S-rescue:Conn_02x10_Odd_Even-Model_S
- J6: footprint Connector_PinHeader_2.54mm:PinHeader_1x06_P2.54mm_Vertical -> Model_S:PinHeader_1x06_P2.54mm_Vertical; symbol Connector_Generic:Conn_01x06 -> Model-S-rescue:Conn_01x06-Model_S
- J7: footprint Connector_PinHeader_2.54mm:PinHeader_1x04_P2.54mm_Vertical -> Model_S:PinHeader_1x04_P2.54mm_Vertical; symbol Connector_Generic:Conn_01x04 -> Model-S-rescue:Conn_01x04-Model_S
- J8: footprint Connector_PinHeader_2.54mm:PinHeader_2x03_P2.54mm_Vertical -> Model_S:PinHeader_2x03_P2.54mm_Vertical; symbol Connector_Generic:Conn_02x03_Odd_Even -> Model-S-rescue:Conn_02x03_Odd_Even-Model_S
- L1: footprint Inductor_SMD:L_0805_2012Metric_Pad1.15x1.40mm_HandSolder -> Model_S:L_0805_2012Metric_Pad1.15x1.40mm_HandSolder; symbol Device:L -> Model-S-rescue:L-Model_S
- Q1: footprint Package_TO_SOT_SMD:SOT-23 -> Model_S:SOT-23; symbol Transistor_FET:BSS138 -> Model-S-rescue:BSS138-Model_S
- R1, R2, R3, R4, R5, R6, R7: footprint Resistor_SMD:R_0805_2012Metric_Pad1.15x1.40mm_HandSolder -> Model_S:R_0805_2012Metric_Pad1.20x1.40mm_HandSolder; symbol Device:R -> Model-S-rescue:R-Model_S
- SW2: footprint Button_Switch_SMD:SW_SPST_TL3342 -> Model_S:SW_SPST_TL3342; symbol Model-S-rescue:SW_PUSH-keyboard_parts -> Model-S-rescue:SW_SPST-Model_S
- U1: footprint GCPCBFootprints:TPS61240 -> Model_S:TPS61240; symbol Model-S-rescue:TPS61240-GCPCBLibrary -> Model-S-rescue:TPS61240-Model_S
- U2: footprint Package_SO:VSSOP-10_3x3mm_P0.5mm -> Model_S:VSSOP-10_3x3mm_P0.5mm; symbol Model-S-rescue:TS3USB30-GCPCBLibrary -> Model-S-rescue:TS3USB30-Model_S
- U3: footprint Package_QFP:TQFP-44_10x10mm_P0.8mm -> Model_S:TQFP-44_10x10mm_P0.8mm; symbol Model-S-rescue:ATmega32U4-AU-MCU_Microchip_ATmega -> Model-S-rescue:32u4-Model_S
- X1: footprint Crystal:Crystal_SMD_TXC_7M-4Pin_3.2x2.5mm -> Model_S:Crystal_SMD_TXC_7M-4Pin_3.2x2.5mm; symbol Model-S-rescue:XTAL_GND-keyboard_parts -> Model-S-rescue:XTAL_GND-Model_S
Other:
- note added: "(5V)"
- note added: "(USB Data)"
- note added: "3.3V"
- note added: "Crane Model S"
- note added: "Data Line Level Shifter"
- note added: "Decoupling\nCapacitors"
- note added: "GC\nData"
- note removed: "Logic Conversion"
- note removed: "Power\nFiltering"

Commit message: Model S 2.2
Parts:
- removed J1: USB_C_Receptacle, Model_S:Shou Han Type-C 24P QCHT, symbol Model-S-rescue:USB_C_Receptacle-Model_S
- removed J6: Debug, Model_S:PinHeader_1x06_P2.54mm_Vertical, symbol Model-S-rescue:Conn_01x06-Model_S
- removed U1: TPS61240, Model_S:TPS61240, symbol Model-S-rescue:TPS61240-Model_S
- added C3, C4, C5: 22uF, Model_S:C_0805_2012Metric_Pad1.18x1.45mm_HandSolder, symbol Model-S-rescue:C_Small-Model_S
- added J1: USB-C Port, Project_Pico:Crane_USBC, symbol Connector_Generic:Conn_02x04_Top_Bottom
- added R1: 402k, Model_S:R_0805_2012Metric_Pad1.20x1.40mm_HandSolder, symbol Model-S-rescue:R-Model_S
- added R2: 100k, Model_S:R_0805_2012Metric_Pad1.20x1.40mm_HandSolder, symbol Model-S-rescue:R-Model_S
- added U1: TPS61230DRC, Package_SON:Texas_S-PVSON-N10_ThermalVias, symbol Regulator_Switching:TPS61230DRC
- C1: value 2.2uF -> 22uF
- C2: value 4.7uF -> 10nF
- L1: footprint Model_S:L_0805_2012Metric_Pad1.15x1.40mm_HandSolder -> Inductor_SMD:L_1008_2520Metric
- renumbered C7 to C10, C8 to C11, C9 to C12, C10 to C13, C12 to C14, C11 to C15, C3 to C6, C4 to C7, C5 to C8, C6 to C9, J7 to J3, J8 to J4, J3 to J5, J5 to J6, J4 to J7, R2 to R3, R3 to R4, R7 to R5, R1 to R6, R4 to R7, R5 to R8, R6 to R9, SW2 to SW1
Connections:
- wire segments 202 -> 221
Other:
- note removed: "(5V)"
- note removed: "(USB Data)"
- note removed: "3.3V"
- note removed: "Debug"
- note removed: "GC\nData"
- moved on the sheet: D1, D2, J6

Commit message: Model S 2.3
Parts:
- removed U2: TS3USB30E, Model_S:VSSOP-10_3x3mm_P0.5mm, symbol Model-S-rescue:TS3USB30-Model_S
- added U2: TS3USB30ERSWR, Model_S:UQFN-10_1.4x1.8mm_P0.4mm, symbol Model-S-rescue:TS3USB30ERSWR-Model_S
Connections:
- net D+: now also U2.3 (D+)
- net D-: now also U2.5 (D-)
- net D1+: now also U2.1 (D1+)
- net D1-: now also U2.7 (D1-)
- net D11: now also U2.10 (S)
- net D2+: now also U2.2 (D2+)
- net D2-: now also U2.6 (D2-)
- net GND: now also U2.4 (GND), U2.8 (OE)
- net VBUS: now also U2.9 (VCC)
Changed lines of the file:
@@
 Sheet 1 1
 Title "Model S"
-Date "2021-07-16"
-Rev "v2.2"
+Date "2021-10-27"
+Rev "v2.3"
 Comp "Crane's Lab"
 Comment1 ""
@@
 	1    0    0    1
 $EndComp
-$Comp
-L Model-S-rescue:TS3USB30-Model_S U2
-U 1 1 5DB586E4
-P 5150 6600
-F 0 "U2" H 4850 6950 50  0000 L CNN
-F 1 "TS3USB30E" V 5150 6450 50  0000 L CNN
-F 2 "Model_S:VSSOP-10_3x3mm_P0.5mm" V 5250 6600 50  0001 C CNN
-F 3 "" V 5250 6600 50  0001 C CNN
-	1    5150 6600
-	1    0    0    -1
-$EndComp
 Text Notes 5900 5950 2    79   ~ 0
 USB Switch
@@
 Wire Wire Line
 	2450 2750 2450 2800
+$Comp
+L Model-S-rescue:TS3USB30ERSWR-Model_S U2
+U 1 1 6149456D
+P 5150 6600
+F 0 "U2" H 4850 6950 50  0000 L CNN
+F 1 "TS3USB30ERSWR" H 5250 7050 50  0000 L CNN
+F 2 "Model_S:UQFN-10_1.4x1.8mm_P0.4mm" V 4500 6600 50  0001 C CNN
+F 3 "" V 4500 6600 50  0001 C CNN
+	1    5150 6600
+	1    0    0    -1
+$EndComp
 $EndSCHEMATC
